Commit message: fix urdf for simulation

File: src/mini_simulation/urdf/accessories/rplidar_s2.urdf (robot description, URDF)
Before this commit: robot rplidar_s2, 1 links, 1 joints
Links:
- link lidar_link: geometry collision mesh filename=file://$(find mini_simulation)/meshes/centered_rplidar-s1m1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 scale=0.001 0.001 0.001; visual mesh filename=file://$(find mini_simulation)/meshes/centered_rplidar-s1m1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 scale=0.001 0.001 0.001

File: src/mini_simulation/urdf/mini.urdf (robot description, URDF)
Before this commit: robot rover_mini, 7 links, 6 joints
Links:
- link chassis_link: geometry collision mesh filename=file://$(find mini_simulation)/meshes/mini_chassis.dae; visual mesh filename=file://$(find mini_simulation)/meshes/mini_chassis.dae
- link fl_wheel_link: geometry collision mesh filename=file://$(find mini_simulation)/meshes/hub_6.5in.dae; visual mesh filename=file://$(find mini_simulation)/meshes/hub_6.5in.dae
- link fr_wheel_link: geometry collision mesh filename=file://$(find mini_simulation)/meshes/hub_6.5in.dae; visual mesh filename=file://$(find mini_simulation)/meshes/hub_6.5in.dae
- link rl_wheel_link: geometry collision mesh filename=file://$(find mini_simulation)/meshes/hub_6.5in.dae; visual mesh filename=file://$(find mini_simulation)/meshes/hub_6.5in.dae
- link rr_wheel_link: geometry collision mesh filename=file://$(find mini_simulation)/meshes/hub_6.5in.dae; visual mesh filename=file://$(find mini_simulation)/meshes/hub_6.5in.dae
